File: 32u4_breakout.kicad_sch (KiCad schematic)
At the start: 15 parts, among them J1 ICSP, J8 PWR, J9 GND, U1 ATmega32U4-A, Y1 16 MHz

Commit message: Added LED for power and PC7/IO13
Parts:
- added D1, D2: LED, LED_SMD:LED_1206_3216Metric, symbol Device:LED
- added R1, R2: 220, Resistor_SMD:R_1206_3216Metric, symbol Device:R
Connections:
- net 5V: now also D1.2 (A)
- net GND: now also R1.2, R2.2
- net IO13: now reaches J6.2 (Pin_2), U1.32 (PC7)
- net IO13: now also D2.2 (A)
- new net: D2.1 (K), R2.1
- new net: D1.1 (K), R1.1
